File: ATmega644.kicad_pcb (KiCad board)
At the start: 2 copper layers, 133 x 110.8 mm, 105 parts, among them J1 PortA_LEDS_en, J10 FTDI, J11 FTDI_VCC_en, J12 FTDI_DTR_en, J13 LCD, J14 Conn_01x02, J15 PORTB, J16 PORTD, J17 Supply, J18 Supply, J19 LCD_Interface, J2 PortB_LEDS_en, J20 Buttons, J21 Power Supply, J3 AVR-ISP-6, J4 PORTA, J5 PORTC, J6 AVR-JTAG-10, J7 Serial, J8 I2C, J9 AVR-JTAG-10, Q1 2N7002, Q10 2N7002, Q11 2N7002, Q12 2N7002, Q13 2N7002, Q14 2N7002, Q15 2N7002, Q16 2N7002, Q17 2N7002, Q2 2N7002, Q3 2N7002, Q4 2N7002, Q5 2N7002, Q6 2N7002, Q7 2N7002, Q8 2N7002, Q9 2N7002, SW1 SW_Push_Open_Dual, SW2 SW_Push_Open_Dual, SW3 SW_Push_Open_Dual, SW4 SW_Push_Open_Dual, SW5 SW_Push_Open_Dual, SW6 SW_Push_Open_Dual, SW7 SW_Push_Open_Dual, SW8 SW_Push_Open_Dual, SW9 SW_Push_Open_Dual, U1 TSR1-2450E, U2 ATmega644-20P, Y1 20 MHz

Commit message: added pix
Other:
- board text added: "ATmega1284p Development Board 2024-10-13 https://github.com/chrisgoertz/ATmega1284p_DevBoard.git"
- board text removed: "ATmega1284p Development Board 2024-10-13 <chris.goertz@gmx.de>"
Changed lines of the file:
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@@
 		)
 	)
-	(gr_text "ATmega1284p Development Board\n2024-10-13\n<chris.goertz@gmx.de>\n"
-		(at 66.75 84.75 270)
+	(gr_text "ATmega1284p Development Board\n2024-10-13\nhttps://github.com/chrisgoertz/ATmega1284p_DevBoard.git\n"
+		(at 65.5 61.5 270)
 		(layer "F.SilkS")
 		(effects
